Commit message: velocity limit

File: delybot_description/urdf/delybot.urdf.xacro (robot description, xacro)
@@ -2,14 +2,14 @@
 <robot xmlns:xacro="http://www.ros.org/wiki/xacro" name="delybot">
     <!-- BOX PROPERTIES -->
-    <xacro:property name="box_width" value="0.61" />
-    <xacro:property name="box_depth" value="0.762" />
-    <xacro:property name="box_height" value="0.737" />
+    <xacro:property name="box_width" value="0.45" />
+    <xacro:property name="box_depth" value="0.63" />
+    <xacro:property name="box_height" value="0.54" />
     <xacro:property name="box_mass" value="42" />
     <!-- WHEEL PROPERTIES -->
-    <xacro:property name="wheel_radius" value="0.08" />
-    <xacro:property name="wheel_width" value="0.03" />
-    <xacro:property name="wheel_offset_from_bottom_chassis" value="0.01" />
-    <xacro:property name="wheel_offset_from_front_chassis" value="0.02" />
-    <xacro:property name="wheel_offset_from_back_chassis" value="0.02" />
+    <xacro:property name="wheel_radius" value="0.11" />
+    <xacro:property name="wheel_width" value="0.08" />
+    <xacro:property name="wheel_offset_from_bottom_chassis" value="0.0" />
+    <xacro:property name="wheel_offset_from_front_chassis" value="0.0" />
+    <xacro:property name="wheel_offset_from_back_chassis" value="0.0" />
     <xacro:property name="wheel_mass" value="0.5" />
     <!-- MACRO DEFINITION -->

Commit message: LIDAR implemented

File: delybot_description/urdf/delybot.urdf.xacro (robot description, xacro)
@@ -34,6 +34,6 @@
                 <origin xyz="0.0 0.0 0.0" rpy="1.57075 0.0 0.0"/>
                 <geometry>
-                   <cylinder radius="${wheel_radius}" length="${wheel_width}"/>
-               </geometry>
+                    <cylinder radius="${wheel_radius}" length="${wheel_width}"/>
+                </geometry>
             </collision>
             <xacro:default_inertial mass="${wheel_mass}"/>
@@ -48,5 +48,5 @@
         </joint>
         <gazebo reference="${position}_wheel">
-            <material>Gazebo/Black</material>
+            <material>Gazebo/FlatBlack</material>
         </gazebo>
         <!-- TRASMISSION DEFINITION -->
@@ -106,5 +106,37 @@
     <!-- RIGHT BACK WHEEL -->
     <xacro:wheel_macro position="right_back" x="${-box_depth/2 + wheel_offset_from_front_chassis}" y="${-box_width/2 - wheel_width/2}"/>
+    <!-- LIDAR SENSOR -->
+    <joint name="scan_joint" type="fixed">
+        <parent link="base_link"/>
+        <child link="base_scan"/>
+        <origin xyz="0 0 ${box_height/2 + 0.0315}" rpy="0 0 0"/>
+    </joint>
+    <link name="base_scan">
+        <visual>
+            <origin xyz="0 0 0" rpy="0 0 0"/>
+                <geometry>
+                    <mesh filename="package://delybot_description/sensors/lds.stl" scale="0.001 0.001 0.001"/>
+                </geometry>
+            <material name="black"/>
+        </visual>
+        <collision>
+            <origin xyz="0.015 0 -0.0065" rpy="0 0 0"/>
+            <geometry>
+                <cylinder length="0.0315" radius="0.055"/>
+            </geometry>
+        </collision>
+        <inertial>
+            <mass value="0.114" />
+            <origin xyz="0 0 0" />
+            <inertia ixx="0.001" ixy="0.0" ixz="0.0"
+                    iyy="0.001" iyz="0.0"
+                    izz="0.001" />
+        </inertial>
+    </link>
+    <gazebo reference="base_scan">
+        <material>Gazebo/FlatBlack</material>
+    </gazebo>
     <!-- GAZEBO PLUGIN -->
+    <!-- ROS CONTROL PLUGIN -->
     <gazebo>
         <plugin name="gazebo_ros_control" filename="libgazebo_ros_control.so">
@@ -112,3 +144,36 @@
         </plugin>
     </gazebo>
+    <!-- LIDAR SENSOR PLUGIN -->
+    <gazebo reference="base_scan">
+        <material>Gazebo/FlatBlack</material>
+        <sensor type="ray" name="lds_lfcd_sensor">
+            <pose>0 0 0 0 0 0</pose>
+            <visualize>true</visualize>
+            <update_rate>5</update_rate>
+            <ray>
+                <scan>
+                    <horizontal>
+                        <samples>360</samples>
+                        <resolution>1</resolution>
+                        <min_angle>0.0</min_angle>
+                        <max_angle>6.28319</max_angle>
+                    </horizontal>
+                </scan>
+                <range>
+                    <min>0.120</min>
+                    <max>3.5</max>
+                    <resolution>0.015</resolution>
+                </range>
+                <noise>
+                    <type>gaussian</type>
+                    <mean>0.0</mean>
+                    <stddev>0.01</stddev>
+                </noise>
+            </ray>
+            <plugin name="gazebo_ros_lds_lfcd_controller" filename="libgazebo_ros_laser.so">
+                <topicName>scan</topicName>
+                <frameName>base_scan</frameName>
+            </plugin>
+        </sensor>
+    </gazebo>
 </robot>

Commit message: IMU implemented

File: delybot_description/urdf/delybot.urdf.xacro (robot description, xacro)
@@ -22,5 +22,5 @@
     </xacro:macro>
     <!-- WHEEL MACRO -->
-    <xacro:macro name="wheel_macro" params="position x y">
+    <xacro:macro name="wheel_macro" params="position x y actuated:=false">
         <link name="${position}_wheel">
             <visual>
@@ -56,8 +56,10 @@
                 <hardwareInterface>hardware_interface/VelocityJointInterface</hardwareInterface>
             </joint>
-            <actuator name="${position}_wheel_joint_motor">
-                <hardwareInterface>hardware_interface/EffortJointInterface</hardwareInterface>
-                <mechanicalReduction>1</mechanicalReduction>
-            </actuator>
+            <xacro:if value="true">
+                <actuator name="${position}_wheel_joint_motor">
+                    <hardwareInterface>hardware_interface/EffortJointInterface</hardwareInterface>
+                    <mechanicalReduction>1</mechanicalReduction>
+                </actuator>
+            </xacro:if>
         </transmission>
     </xacro:macro>
@@ -95,20 +97,20 @@
     </joint>
     <!-- LEFT FRONT WHEEL -->
-    <xacro:wheel_macro position="left_front" x="${box_depth/2 - wheel_offset_from_front_chassis}" y="${box_width/2 + wheel_width/2}"/>
+    <xacro:wheel_macro position="left_front" x="${box_depth/2 - wheel_offset_from_front_chassis}" y="${box_width/2 + wheel_width/2}" actuated="true"/>
     <!-- LEFT CENTER WHEEL -->
     <xacro:wheel_macro position="left_center" x="0" y="${box_width/2 + wheel_width/2}"/>
     <!-- LEFT BACK WHEEL -->
-    <xacro:wheel_macro position="left_back" x="${-box_depth/2 + wheel_offset_from_front_chassis}" y="${box_width/2 + wheel_width/2}"/>
+    <xacro:wheel_macro position="left_back" x="${-box_depth/2 + wheel_offset_from_front_chassis}" y="${box_width/2 + wheel_width/2}" actuated="true"/>
     <!-- RIGHT FRONT WHEEL -->
-    <xacro:wheel_macro position="right_front" x="${box_depth/2 - wheel_offset_from_front_chassis}" y="${-box_width/2 - wheel_width/2}"/>
+    <xacro:wheel_macro position="right_front" x="${box_depth/2 - wheel_offset_from_front_chassis}" y="${-box_width/2 - wheel_width/2}" actuated="true"/>
     <!-- RIGHT CENTER WHEEL -->
     <xacro:wheel_macro position="right_center" x="0" y="${-box_width/2 - wheel_width/2}"/>
     <!-- RIGHT BACK WHEEL -->
-    <xacro:wheel_macro position="right_back" x="${-box_depth/2 + wheel_offset_from_front_chassis}" y="${-box_width/2 - wheel_width/2}"/>
+    <xacro:wheel_macro position="right_back" x="${-box_depth/2 + wheel_offset_from_front_chassis}" y="${-box_width/2 - wheel_width/2}" actuated="true"/>
     <!-- LIDAR SENSOR -->
     <joint name="scan_joint" type="fixed">
         <parent link="base_link"/>
         <child link="base_scan"/>
-        <origin xyz="0 0 ${box_height/2 + 0.0315}" rpy="0 0 0"/>
+        <origin xyz="${box_depth/4} 0 ${box_height/2 + 0.0315}" rpy="0 0 0"/>
     </joint>
     <link name="base_scan">
@@ -137,4 +139,11 @@
         <material>Gazebo/FlatBlack</material>
     </gazebo>
+    <!-- IMU SENSOR -->
+    <link name="imu_link"/>
+    <joint name="imu_joint" type="fixed">
+        <parent link="base_link"/>
+        <child link="imu_link"/>
+        <origin xyz="0.0 0 ${box_height/2}" rpy="0 0 0"/>
+    </joint>
     <!-- GAZEBO PLUGIN -->
     <!-- ROS CONTROL PLUGIN -->
@@ -162,5 +171,5 @@
                 <range>
                     <min>0.120</min>
-                    <max>3.5</max>
+                    <max>5</max>
                     <resolution>0.015</resolution>
                 </range>
@@ -177,3 +186,39 @@
         </sensor>
     </gazebo>
+    <!-- IMU PLUGIN -->
+    <gazebo reference="imu_link">
+        <sensor type="imu" name="imu">
+            <always_on>true</always_on>
+            <visualize>true</visualize>
+        </sensor>
+        <material>Gazebo/Grey</material>
+    </gazebo>
+    <gazebo>
+    <plugin name="imu_plugin" filename="libgazebo_ros_imu.so">
+        <alwaysOn>true</alwaysOn>
+        <bodyName>imu_link</bodyName>
+        <frameName>imu_link</frameName>
+        <topicName>imu</topicName>
+        <serviceName>imu_service</serviceName>
+        <gaussianNoise>0.0</gaussianNoise>
+        <updateRate>0</updateRate>
+        <imu>
+        <noise>
+            <type>gaussian</type>
+                <rate>
+                    <mean>0.0</mean>
+                    <stddev>2e-4</stddev>
+                    <bias_mean>0.0000075</bias_mean>
+                     <bias_stddev>0.0000008</bias_stddev>
+                </rate>
+                    <accel>
+                       <mean>0.0</mean>
+                        <stddev>1.7e-2</stddev>
+                        <bias_mean>0.1</bias_mean>
+                        <bias_stddev>0.001</bias_stddev>
+                    </accel>
+                </noise>
+            </imu>
+        </plugin>
+    </gazebo>
 </robot>

Commit message: Fixed robot rotation

File: delybot_description/urdf/delybot.urdf.xacro (robot description, xacro)
@@ -12,5 +12,5 @@
     <xacro:property name="wheel_offset_from_front_chassis" value="0.05" />
     <xacro:property name="wheel_offset_from_back_chassis" value="0.05" />
-    <xacro:property name="wheel_mass" value="0.01" />    <!-- original: 0.5 kg-->
+    <xacro:property name="wheel_mass" value="0.5" />    <!-- original: 0.5 kg-->
     <!-- MACRO DEFINITION -->
     <!-- DEFAULT INERTIA MACRO -->
@@ -65,5 +65,5 @@
             <!-- <mu1 value="100.0"/>
             <mu2 value="50.0"/> -->
-            <kp value="1000000.0" />     <!-- 500000 -->
+            <kp value="1000000.0" />
             <kd value="1.0" />
             <selfCollide>true</selfCollide>
@@ -88,5 +88,5 @@
             <xacro:if value="true">
                 <actuator name="${position}_wheel_joint_motor">
-                    <hardwareInterface>hardware_interface/VelocityJointInterface</hardwareInterface>
+                    <hardwareInterface>hardware_interface/EffortJointInterface</hardwareInterface>
                     <mechanicalReduction>1</mechanicalReduction>
                 </actuator>
@@ -130,5 +130,5 @@
     <xacro:wheel_macro position="left_front" x="${box_depth/2 - wheel_offset_from_front_chassis}" y="${box_width/2 + wheel_width/2}" actuated="true"/>
     <!-- LEFT CENTER WHEEL -->
-    <!-- <xacro:wheel_macro position="left_center" x="0" y="${box_width/2 + wheel_width/2}"/> -->
+    <xacro:wheel_macro position="left_center" x="0" y="${box_width/2 + wheel_width/2}"/>
     <!-- LEFT BACK WHEEL -->
     <xacro:wheel_macro position="left_back" x="${-box_depth/2 + wheel_offset_from_front_chassis}" y="${box_width/2 + wheel_width/2}" actuated="true"/>
@@ -136,5 +136,5 @@
     <xacro:wheel_macro position="right_front" x="${box_depth/2 - wheel_offset_from_front_chassis}" y="${-box_width/2 - wheel_width/2}" actuated="true"/>
     <!-- RIGHT CENTER WHEEL -->
-    <!-- <xacro:wheel_macro position="right_center" x="0" y="${-box_width/2 - wheel_width/2}"/> -->
+    <xacro:wheel_macro position="right_center" x="0" y="${-box_width/2 - wheel_width/2}"/>
     <!-- RIGHT BACK WHEEL -->
     <xacro:wheel_macro position="right_back" x="${-box_depth/2 + wheel_offset_from_front_chassis}" y="${-box_width/2 - wheel_width/2}" actuated="true"/>
